Commit message: added camera sensor simulation

File: urdf/custom_bot.urdf (robot description, URDF)
Before this commit: robot gbot, 6 links, 5 joints
Links:
- added link camera_link, mass 1e-5; collision box size=0.07 0.07 0.07; visual box size=0.07 0.07 0.07
- added link imu_link, mass 1e-5; collision box size=0.1 0.1 0.1; visual box size=0.1 0.1 0.1
Joints:
- added joint camera_joint: type fixed, parent base_link, child camera_link, origin xyz=0 0 0.15 rpy=0 0 0, axis 0 1 0
- added joint imu_joint: type fixed, parent base_link, child imu_link, origin xyz=-0.3 0.0 0.08 rpy=0 0 0, axis 0 0 0
