Commit message: restructured

File: janky_simulator/urdf/janky_bot.urdf (robot description, URDF)
Before this commit: robot gbot, 8 links, 7 joints
Links:
- added link base_footprint
Joints:
- added joint base_link_joint: type fixed, parent base_footprint, child base_link, origin xyz=-0.2 0.0 -0.2 rpy=0.0 0.0 0.0
- joint camera_joint: origin xyz=0 0 0.15 rpy=0 0 0 -> xyz=0 0 0.15 rpy=0 0.3 0
- joint imu_joint: origin xyz=-0.3 0.0 0.08 rpy=0 0 0 -> xyz=-0.2 0.0 0.08 rpy=0.0 0.0 0.0
